File: Hardware/PCB/usb_rfid_reader/usb_rfid_reader.kicad_pcb (KiCad board)
At the start: 4 copper layers, 90 x 90 mm, 35 parts, among them J1 629722000214, J2 Conn_01x08, J3 Conn_ST_STDC14, Q1 2N3904, SW1 BOOT0, SW2 RESET, U1 AZ1117CH2-3.3, U2 USBLC6-2SC6, U3 STM32L476RGTx

Commit message: ajout modèle 3D socle + dernière modif PCB
Routing:
- net /USER_LED: track 28.3 -> 27.1 mm
Changed lines of the file:
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@@
 	)
 	(segment
-		(start 105.675 67.925)
-		(end 106.449999 67.925)
+		(start 107.18 66.45)
+		(end 115.7 66.45)
 		(width 0.2)
 		(layer "F.Cu")
@@
 	)
 	(segment
-		(start 107.3 66.33)
-		(end 121.4 66.33)
+		(start 106.97 66.66)
+		(end 107.18 66.45)
+		(width 0.2)
+		(layer "F.Cu")
+		(net 33)
+	)
+	(segment
+		(start 115.7 66.45)
+		(end 124.3 75.05)
+		(width 0.2)
+		(layer "F.Cu")
+		(net 33)
+	)
+	(segment
+		(start 106.449999 67.925)
+		(end 106.97 67.404999)
+		(width 0.2)
+		(layer "F.Cu")
+		(net 33)
+	)
+	(segment
+		(start 105.675 67.925)
+		(end 106.449999 67.925)
 		(width 0.2)
 		(layer "F.Cu")
@@
 	)
 	(segment
-		(start 106.449999 67.925)
-		(end 106.97 67.404999)
-		(width 0.2)
-		(layer "F.Cu")
-		(net 33)
-	)
-	(segment
-		(start 121.4 66.33)
-		(end 128.175 73.105)
-		(width 0.2)
-		(layer "F.Cu")
-		(net 33)
-	)
-	(segment
-		(start 106.97 66.66)
-		(end 107.3 66.33)
-		(width 0.2)
-		(layer "F.Cu")
-		(net 33)
-	)
-	(segment
-		(start 128.175 73.105)
+		(start 124.3 75.05)
 		(end 128.175 75.05)
 		(width 0.2)

Commit message: ajout des fichier gerber
Parts:
- removed Q1: 2N3904, Package_TO_SOT_THT:TO-92_Inline
- added Q2: NMOS, Package_TO_SOT_SMD:SOT-23-3, F.Cu at (114.3, 64.3)
- added R8: 1k, Resistor_SMD:R_0603_1608Metric, F.Cu at (114.6, 61.8)
- added TP1: TestPoint, TestPoint:TestPoint_Pad_D1.0mm, F.Cu at (89.3, 60.5)
- added TP2: TestPoint, TestPoint:TestPoint_Pad_D1.0mm, F.Cu at (87.3, 60.5)
- added TP3: TestPoint, TestPoint:TestPoint_Pad_D1.0mm, F.Cu at (110.8, 64.8)
- added TP4: TestPoint, TestPoint:TestPoint_Pad_D1.0mm, F.Cu at (78.5, 75.0)
- added TP5: TestPoint, TestPoint:TestPoint_Pad_D1.0mm, F.Cu at (78.5, 77.5)
- added TP6: TestPoint, TestPoint:TestPoint_Pad_D1.0mm, F.Cu at (78.5, 80.0)
- added TP7: TestPoint, TestPoint:TestPoint_Pad_D1.0mm, F.Cu at (78.5, 82.5)
- added TP8: TestPoint, TestPoint:TestPoint_Pad_D1.0mm, F.Cu at (78.5, 85.0)
- SW1: value BOOT0 -> RESET
- moved C11 42.4 mm to (123.1, 50.0), turned to -90 degrees
- moved C2 19.0 mm to (85.8, 72.9), turned to 180 degrees
- moved R7 2.67 mm to (92.0, 67.8), turned to -90 degrees
- moved C5 1.17 mm to (90.7, 70.2)
- moved C8 0.72 mm to (108.7, 68.2)
Routing:
- net /RC522_SPI2_CE_N: track 23.4 -> 56.7 mm
- net /RC522_SPI2_CLK: track 21.9 -> 53.4 mm
- net /RC522_RST: track 32.3 -> 47.9 mm, vias 3 -> 1
- net /RC522_SPI2_MISO: track 34.8 -> 45.8 mm, vias 3 -> 1
- net /RC522_SPI2_MOSI: track 42.8 -> 48.4 mm, vias 3 -> 1
- net +3.3V: track 38.9 -> 43.2 mm, vias 15 -> 16
- net /VCP_USART2_RX: track 50.8 -> 47.1 mm
- net /BOOT0: track 37.3 -> 33.7 mm
- net Net-(Q2-G): track 2.98 -> 6.31 mm
- net /NRST: track 97.4 -> 94.3 mm, vias 3 -> 2
- net +5V: track 30.0 -> 33.0 mm
- net /BUZZ_TIM1: track 14.9 -> 17.4 mm
- net Net-(BZ1--): track 12.3 -> 11.1 mm
- net GND: track 24.0 -> 23.0 mm, vias 156 -> 170
- net /USER_LED: track 27.1 -> 26.1 mm
