File: Hardware/PCB/usb_rfid_reader/usb_rfid_reader.kicad_sch (KiCad schematic)
At the start: 35 parts, among them J1 Conn_01x08, J2 Conn_ST_STDC14, J3 10172013-00011LF, Q1 2N3904, SW1 RESET, U1 STM32L476RGTx, U2 AZ1117CH2-3.3, U3 USBLC6-2P6

Commit message: review schematic
Parts:
- removed J3: 10172013-00011LF, 10172013-00011LF:AMPHENOL_10172013-00011LF, symbol 10172013-00011LF:10172013-00011LF
- removed R1, R2: 22, Resistor_SMD:R_0603_1608Metric, symbol Device:R
- removed R3, R4: 5.1k, Resistor_SMD:R_0603_1608Metric, symbol Device:R
- removed U3: USBLC6-2P6, Package_TO_SOT_SMD:SOT-666, symbol Power_Protection:USBLC6-2P6
- added C2: 1u, Capacitor_SMD:C_0603_1608Metric, symbol Device:C
- added J1: 629722000214, Connector_USB:USB_C_Receptacle_HRO_TYPE-C-31-M-12, symbol Connector:USB_C_Receptacle_USB2.0_16P
- added R2, R3: 5k1, Resistor_SMD:R_0402_1005Metric, symbol Device:R_Small
- added SW1: RESET, Button_Switch_SMD:SW_SPST_PTS645Sx43SMTR92, symbol Switch:SW_Push
- added U2: USBLC6-2SC6, Package_TO_SOT_SMD:SOT-23-6, symbol Power_Protection:USBLC6-2SC6
- C10: value 100n -> 10n
- D1, D2, D3: MPN 150060RS75000 -> 150060RS55040
- R4: renamed from R5; value 3k -> 680R
- R5: renamed from R6; value 1.5k -> 300R
- R6: renamed from R9; value 1.5k -> 300R
- renumbered C3 to C11, C2 to C3, J1 to J2, J2 to J3, R8 to R1, SW1 to SW2, U2 to U1, U1 to U3
Connections:
- net +3.3V: now also C2.1, SW1.1
- net +5V: now also J1.A4 (VBUS), J1.A9 (VBUS), J1.B4 (VBUS), J1.B9 (VBUS), U2.5 (VBUS)
- net D+: now also J1.A6 (D+), J1.B6 (D+), U2.6 (I/O1)
- net D-: now also J1.A7 (D-), J1.B7 (D-), U2.4 (I/O2)
- net GND: now also C2.2, J1.A1 (GND), J1.A12 (GND), J1.B1 (GND), J1.B12 (GND), J1.S1 (SHIELD), R2.1, R3.2, U2.2 (GND)
- net SPI2_RST: no longer J2.2 (Pin_2)
- net USART2_RX: now also J3.13 (VCP_RX); no longer J3.14 (VCP_TX)
- net USART2_TX: now also J3.14 (VCP_TX); no longer J3.13 (VCP_RX)
- net USB_DM: now also U2.3 (I/O2)
- net USB_DP: now also U2.1 (I/O1)
- net BOOT0: now reaches R7.2, U3.60 (BOOT0)
- net BOOT0: now also SW1.2
- net RC522_SPI2_CE_N: now reaches U3.33 (PB12)
- net RC522_SPI2_CE_N: now also J2.8 (Pin_8)
- net RC522_SPI2_CLK: now reaches U3.34 (PB13)
- net RC522_SPI2_CLK: now also J2.7 (Pin_7)
- net RC522_SPI2_MISO: now reaches U3.35 (PB14)
- net RC522_SPI2_MISO: now also J2.5 (Pin_5)
- net RC522_SPI2_MOSI: now reaches U3.36 (PB15)
- net RC522_SPI2_MOSI: now also J2.6 (Pin_6)
- net RC522_RST: now reaches U3.37 (PC6)
- net RC522_RST: now also J2.2 (Pin_2)
- net BUZZ renamed BUZZ_TIM1
- net SPI2_MISO: no longer names the net of U3.10 (PC2)
- net SPI2_MISO: no longer J2.5 (Pin_5)
- net SPI2_MOSI: no longer names the net of U3.11 (PC3)
- net SPI2_MOSI: no longer J2.6 (Pin_6)
- net SPI2_SCK: no longer names the net of U3.29 (PB10)
- net SPI2_SCK: no longer J2.7 (Pin_7)
- net SPI2_SDA: no longer names the net of U3.14 (PA0)
- net SPI2_SDA: no longer J2.8 (Pin_8)
- new net: J1.A5 (CC1), R2.2
- new net: J1.B5 (CC2), R3.1
- no-connect marks 43 -> 41
Other:
- note added: "1.8V @ 5mA"
- note added: "Connecteur USB-C : Data + 5V"
- note added: "RFID"
- note removed: "Connecteur SPI + STlink"
- note removed: "Connecteur USB-C"
- note removed: "Powerflag"
- moved on the sheet: BZ1, C1, C10, C11, C3, C4, C5, C6, C7, C8, C9, D1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

Commit message: corrections schéma
Connections:
- net SPI2_RST: no longer names the net of U3.15 (PA1)
- net USART2_RX renamed VCP_USART2_RX
- net USART2_TX renamed VCP_USART2_TX
- no-connect marks 41 -> 42
Other:
- moved on the sheet: H1

Commit message: modification classes jango
Parts:
- J1: footprint Connector_USB:USB_C_Receptacle_HRO_TYPE-C-31-M-12 -> 10172013-00011LF:AMPHENOL_10172013-00011LF
Changed lines of the file:
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@@
 			)
 		)
-		(property "Footprint" "Connector_USB:USB_C_Receptacle_HRO_TYPE-C-31-M-12"
+		(property "Footprint" "10172013-00011LF:AMPHENOL_10172013-00011LF"
 			(at 48.26 45.72 0)
 			(effects

Commit message: routage PCB avant ERC
Parts:
- C1: MPN GRM188R61A106KE69D -> 885012106031
- C3: MPN GRM21BR61A226ME44L -> 865060442002
- J1: footprint 10172013-00011LF:AMPHENOL_10172013-00011LF -> Connector_USB:USB_C_Receptacle_HRO_TYPE-C-31-M-12
- renumbered R2 to R1, R3 to R2, R1 to R3
Connections:
- net USER_LED: now also U3.22 (PA6); no longer U3.40 (PC9)
Changed lines of the file:
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@@
 	)
 	(no_connect
+		(at 158.75 104.14)
+	)
+	(no_connect
 		(at 158.75 76.2)
 	)
@@
 	)
 	(no_connect
-		(at 194.31 73.66)
-	)
-	(no_connect
 		(at 194.31 101.6)
 	)
@@
 	(wire
 		(pts
+			(xy 194.31 73.66) (xy 209.55 73.66)
+		)
+		(stroke
+			(width 0)
+			(type default)
+		)
+	)
+	(wire
+		(pts
 			(xy 194.31 66.04) (xy 198.12 66.04)
 		)
@@
 	(wire
 		(pts
-			(xy 149.86 104.14) (xy 158.75 104.14)
-		)
-		(stroke
-			(width 0)
-			(type default)
-		)
-	)
-	(wire
-		(pts
 			(xy 107.95 44.45) (xy 109.22 44.45)
 		)
@@
 		)
 	)
-	(label "RC522_RST"
-		(at 213.36 46.99 0)
-		(effects
-			(font
-				(size 1.27 1.27)
-			)
-			(justify left bottom)
-		)
-	)
 	(label "NRST"
 		(at 151.13 58.42 0)
@@
 		)
 	)
+	(label "USER_LED"
+		(at 209.55 73.66 180)
+		(effects
+			(font
+				(size 1.27 1.27)
+			)
+			(justify right bottom)
+		)
+	)
 	(label "RC522_SPI2_MISO"
 		(at 213.36 137.16 180)
@@
 		)
 	)
-	(label "USER_LED"
-		(at 149.86 104.14 180)
-		(effects
-			(font
-				(size 1.27 1.27)
-			)
-			(justify right bottom)
-		)
-	)
 	(label "RC522_SPI2_CLK"
 		(at 40.64 182.88 0)
@@
 		(dnp no)
 		(fields_autoplaced yes)
-		(property "Reference" "#PWR08"
+		(property "Reference" "#PWR013"
 			(at 59.69 151.13 0)
 			(effects
@@
 			(project "usb_rfid_reader"
 				(path "/4e7c00f6-ef26-450d-ba16-3b994e0b74e3"
-					(reference "#PWR08")
+					(reference "#PWR013")
 					(unit 1)
 				)
@@
 		(on_board yes)
 		(dnp no)
-		(property "Reference" "#PWR030"
+		(property "Reference" "#PWR031"
 			(at 243.84 63.5 0)
 			(effects
@@
 			(project "usb_rfid_reader"
 				(path "/4e7c00f6-ef26-450d-ba16-3b994e0b74e3"
-					(reference "#PWR030")
+					(reference "#PWR031")
 					(unit 1)
 				)
@@
 		(dnp no)
 		(fields_autoplaced yes)
-		(property "Reference" "#PWR013"
+		(property "Reference" "#PWR011"
 			(at 59.69 74.93 0)
 			(effects
@@
 			(project "usb_rfid_reader"
 				(path "/4e7c00f6-ef26-450d-ba16-3b994e0b74e3"
-					(reference "#PWR013")
+					(reference "#PWR011")
 					(unit 1)
 				)
@@
 		(on_board yes)
 		(dnp no)
-		(property "Reference" "#PWR025"
+		(property "Reference" "#PWR026"
 			(at 177.8 53.34 0)
 			(effects
@@
 			(project "usb_rfid_reader"
 				(path "/4e7c00f6-ef26-450d-ba16-3b994e0b74e3"
-					(reference "#PWR025")
+					(reference "#PWR026")
 					(unit 1)
 				)
@@
 		(on_board yes)
 		(dnp no)
-		(property "Reference" "R2"
+		(property "Reference" "R1"
 			(at 30.48 33.528 90)
 			(effects
@@
 			(project "usb_rfid_reader"
 				(path "/4e7c00f6-ef26-450d-ba16-3b994e0b74e3"
-					(reference "R2")
+					(reference "R1")
 					(unit 1)
 				)
@@
 		(dnp no)
 		(fields_autoplaced yes)
-		(property "Reference" "#PWR09"
+		(property "Reference" "#PWR07"
 			(at 45.72 104.14 0)
 			(effects
@@
 			(project "usb_rfid_reader"
 				(path "/4e7c00f6-ef26-450d-ba16-3b994e0b74e3"
-					(reference "#PWR09")
+					(reference "#PWR07")
 					(unit 1)
 				)
@@
 		(dnp no)
 		(fields_autoplaced yes)
-		(property "Reference" "#PWR031"
+		(property "Reference" "#PWR032"
 			(at 259.08 134.62 0)
 			(effects
@@
 			(project "usb_rfid_reader"
 				(path "/4e7c00f6-ef26-450d-ba16-3b994e0b74e3"
-					(reference "#PWR031")
+					(reference "#PWR032")
 					(unit 1)
 				)
@@
 		(dnp no)
 		(fields_autoplaced yes)
-		(property "Reference" "#PWR011"
+		(property "Reference" "#PWR010"
 			(at 52.07 172.72 0)
 			(effects
@@
 			(project "usb_rfid_reader"
 				(path "/4e7c00f6-ef26-450d-ba16-3b994e0b74e3"
-					(reference "#PWR011")
+					(reference "#PWR010")
 					(unit 1)
 				)
@@
 		(dnp no)
 		(fields_autoplaced yes)
-		(property "Reference" "#PWR010"
+		(property "Reference" "#PWR09"
 			(at 54.61 171.45 0)
 			(effects
@@
 			(project "usb_rfid_reader"
 				(path "/4e7c00f6-ef26-450d-ba16-3b994e0b74e3"
-					(reference "#PWR010")
+					(reference "#PWR09")
 					(unit 1)
 				)
@@
 		(on_board yes)
 		(dnp no)
-		(property "Reference" "R1"
+		(property "Reference" "R3"
 			(at 46.482 141.986 90)
 			(effects
@@
 			(project "usb_rfid_reader"
 				(path "/4e7c00f6-ef26-450d-ba16-3b994e0b74e3"
-					(reference "R1")
+					(reference "R3")
 					(unit 1)
 				)
@@
 		(dnp no)
 		(fields_autoplaced yes)
-		(property "Reference" "#PWR026"
+		(property "Reference" "#PWR027"
 			(at 177.8 153.67 0)
 			(effects
@@
 			(project "usb_rfid_reader"
 				(path "/4e7c00f6-ef26-450d-ba16-3b994e0b74e3"
-					(reference "#PWR026")
+					(reference "#PWR027")
 					(unit 1)
 				)
@@
 		(dnp no)
 		(fields_autoplaced yes)
-		(property "Reference" "#PWR07"
+		(property "Reference" "#PWR012"
 			(at 63.5 129.54 0)
 			(effects
@@
 			(project "usb_rfid_reader"
 				(path "/4e7c00f6-ef26-450d-ba16-3b994e0b74e3"
-					(reference "#PWR07")
+					(reference "#PWR012")
 					(unit 1)
 				)
@@
 		(dnp no)
 		(fields_autoplaced yes)
-		(property "Reference" "#PWR032"
+		(property "Reference" "#PWR023"
 			(at 130.81 191.77 0)
 			(effects
@@
 			(project ""
 				(path "/4e7c00f6-ef26-450d-ba16-3b994e0b74e3"
-					(reference "#PWR032")
+					(reference "#PWR023")
 					(unit 1)
 				)
@@
 		(dnp no)
 		(fields_autoplaced yes)
-		(property "Reference" "#PWR024"
+		(property "Reference" "#PWR025"
 			(at 152.4 41.91 0)
 			(effects
@@
 			(project "usb_rfid_reader"
 				(path "/4e7c00f6-ef26-450d-ba16-3b994e0b74e3"
-					(reference "#PWR024")
+					(reference "#PWR025")
 					(unit 1)
 				)
@@
 		(dnp no)
 		(fields_autoplaced yes)
-		(property "Reference" "#PWR028"
+		(property "Reference" "#PWR029"
 			(at 227.33 140.97 0)
 			(effects
@@
 			(project "usb_rfid_reader"
 				(path "/4e7c00f6-ef26-450d-ba16-3b994e0b74e3"
-					(reference "#PWR028")
+					(reference "#PWR029")
 					(unit 1)
 				)
@@
 		(dnp no)
 		(fields_autoplaced yes)
-		(property "Reference" "#PWR023"
+		(property "Reference" "#PWR024"
 			(at 152.4 26.67 0)
 			(effects
@@
 			(project "usb_rfid_reader"
 				(path "/4e7c00f6-ef26-450d-ba16-3b994e0b74e3"
-					(reference "#PWR023")
+					(reference "#PWR024")
 					(unit 1)
 				)
@@
 			)
 		)
-		(property "MPN" "GRM21BR61A226ME44L"
+		(property "MPN" "865060442002"
 			(at 49.53 107.95 0)
 			(effects
@@
 		(dnp no)
 		(fields_autoplaced yes)
-		(property "Reference" "#PWR027"
+		(property "Reference" "#PWR028"
 			(at 227.33 116.84 0)
 			(effects
@@
 			(project "usb_rfid_reader"
 				(path "/4e7c00f6-ef26-450d-ba16-3b994e0b74e3"
-					(reference "#PWR027")
+					(reference "#PWR028")
 					(unit 1)
 				)
@@
 		(dnp no)
 		(fields_autoplaced yes)
-		(property "Reference" "#PWR012"
+		(property "Reference" "#PWR08"
 			(at 52.07 74.93 0)
 			(effects
@@
 			(project "usb_rfid_reader"
 				(path "/4e7c00f6-ef26-450d-ba16-3b994e0b74e3"
-					(reference "#PWR012")
+					(reference "#PWR08")
 					(unit 1)
 				)
@@
 			)
 		)
-		(property "MPN" "GRM188R61A106KE69D"
+		(property "MPN" "885012106031"
 			(at 24.13 107.95 0)
 			(effects
@@
 		(on_board yes)
 		(dnp no)
-		(property "Reference" "R3"
+		(property "Reference" "R2"
 			(at 30.48 40.132 90)
 			(effects
@@
 			(project "usb_rfid_reader"
 				(path "/4e7c00f6-ef26-450d-ba16-3b994e0b74e3"
-					(reference "R3")
+					(reference "R2")
 					(unit 1)
 				)
@@
 			)
 		)
-		(property "Footprint" "10172013-00011LF:AMPHENOL_10172013-00011LF"
+		(property "Footprint" "Connector_USB:USB_C_Receptacle_HRO_TYPE-C-31-M-12"
 			(at 48.26 45.72 0)
 			(effects
@@
 		(on_board yes)
 		(dnp no)
-		(property "Reference" "#PWR029"
+		(property "Reference" "#PWR030"
 			(at 242.57 101.6 0)
 			(effects
@@
 			(project "usb_rfid_reader"
 				(path "/4e7c00f6-ef26-450d-ba16-3b994e0b74e3"
-					(reference "#PWR029")
+					(reference "#PWR030")
 					(unit 1)
 				)

Commit message: ajout des fichier gerber
Parts:
- removed Q1: 2N3904, Package_TO_SOT_THT:TO-92_Inline, symbol Transistor_BJT:2N3904
- added Q2: NMOS, Package_TO_SOT_SMD:SOT-23-3, symbol Simulation_SPICE:NMOS
- added R8: 1k, Resistor_SMD:R_0603_1608Metric, symbol Device:R
- added TP1, TP2, TP3, TP4, TP5, TP6, TP7, TP8: TestPoint, TestPoint:TestPoint_Pad_D1.0mm, symbol Connector:TestPoint
Connections:
- net +3.3V: now also TP2.1
- net +5V: now also TP1.1
- net BUZZ_TIM1: now also TP3.1
- net GND: now also Q2.3 (S), R8.1
- net RC522_RST: now also TP4.1
- net RC522_SPI2_CE_N: now also TP8.1
- net RC522_SPI2_CLK: now also TP7.1
- net RC522_SPI2_MISO: now also TP5.1
- net RC522_SPI2_MOSI: now also TP6.1
- net at BZ1.2 (-): now also Q2.1 (D)
- net at R3.2: now also Q2.2 (G), R8.2
Other:
- moved on the sheet: BZ1, C2, J2, R3
